File: EL-A0001-00500 - Telemetria Frontal - ALT/EL-A0001-00500 - Telemetria Frontal - ALT/_autosave-EL-A0001-00500 - Telemetria Frontal - ALT.kicad_sch (KiCad schematic)
At the start: 31 parts, among them J1 1-776087-1, J2 UART, U1 YAAJ_BluePill, U2 MP1584, U3 TJA1050-Module, U4 LM324, U5 LM324

Commit message: MOD: placa de telemetria frontal ALT
Parts:
- gave numbers to parts that had none: 2
Changed lines of the file:
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@@
   (symbol (lib_id "power:GND") (at 145.415 62.23 0) (unit 1)
     (in_bom yes) (on_board yes) (fields_autoplaced)
-    (property "Reference" "#PWR?" (id 0) (at 145.415 68.58 0)
+    (property "Reference" "#PWR0117" (id 0) (at 145.415 68.58 0)
       (effects (font (size 1.27 1.27)) hide)
     )
@@
   (symbol (lib_id "Device:C_Small") (at 122.555 135.89 90) (unit 1)
     (in_bom yes) (on_board yes) (fields_autoplaced)
-    (property "Reference" "C?" (id 0) (at 122.5613 130.6281 90))
+    (property "Reference" "C1" (id 0) (at 122.5613 130.6281 90))
     (property "Value" "" (id 1) (at 122.5613 133.165 90))
     (property "Footprint" "" (id 2) (at 122.555 135.89 0)
@@
   (symbol (lib_id "Device:C_Small") (at 137.795 60.325 90) (unit 1)
     (in_bom yes) (on_board yes) (fields_autoplaced)
-    (property "Reference" "C?" (id 0) (at 137.8013 55.0631 90))
+    (property "Reference" "C2" (id 0) (at 137.8013 55.0631 90))
     (property "Value" "100nF" (id 1) (at 137.8013 57.6 90))
     (property "Footprint" "Capacitor_THT:C_Disc_D3.0mm_W2.0mm_P2.50mm" (id 2) (at 137.795 60.325 0)
@@
   (symbol (lib_id "power:GND") (at 130.81 137.795 0) (unit 1)
     (in_bom yes) (on_board yes) (fields_autoplaced)
-    (property "Reference" "#PWR?" (id 0) (at 130.81 144.145 0)
+    (property "Reference" "#PWR0116" (id 0) (at 130.81 144.145 0)
       (effects (font (size 1.27 1.27)) hide)
     )
@@
       (reference "#PWR0115") (unit 1) (value "GND") (footprint "")
     )
+    (path "/f8aac905-c94d-4bcb-952e-1c5c3776e857"
+      (reference "#PWR0116") (unit 1) (value "GND") (footprint "")
+    )
     (path "/30bfa64d-761b-4732-997d-bd4590e66c7b"
-      (reference "#PWR?") (unit 1) (value "GND") (footprint "")
-    )
-    (path "/f8aac905-c94d-4bcb-952e-1c5c3776e857"
-      (reference "#PWR?") (unit 1) (value "GND") (footprint "")
+      (reference "#PWR0117") (unit 1) (value "GND") (footprint "")
     )
     (path "/4bd1e1bf-c0c6-4901-bac9-5a11f3ae27ed"
-      (reference "C?") (unit 1) (value "100nF") (footprint "Capacitor_THT:C_Disc_D3.0mm_W2.0mm_P2.50mm")
+      (reference "C1") (unit 1) (value "100nF") (footprint "Capacitor_THT:C_Disc_D3.0mm_W2.0mm_P2.50mm")
     )
     (path "/dd25d964-e865-42e7-8ad7-bf5fa7f0278a"
-      (reference "C?") (unit 1) (value "100nF") (footprint "Capacitor_THT:C_Disc_D3.0mm_W2.0mm_P2.50mm")
+      (reference "C2") (unit 1) (value "100nF") (footprint "Capacitor_THT:C_Disc_D3.0mm_W2.0mm_P2.50mm")
     )
     (path "/69ed3c2c-eca2-43d3-a0ce-4fcde1c400a3"
