File: EL-A0001-00301-AA - Placa de Fusíveis (Geral)/EL-A0001-00301-AA - Placa de Fusíveis (Geral)/EL-A0001-00301-AA - Placa de Fusíveis (Geral).kicad_pcb (KiCad board)
At the start: 2 copper layers, 20 parts, among them J1 1-776087-1, J2 BUCK_SHUT, J3 SPLIT_POWER, J4 DC_CONVERTER, J5 VBAT

Commit message: AA
Routing:
- added copper zone on B.Cu, net GND
- added copper zone on F.Cu, net GND
Other:
- board outline added: 94.5 x 95.5 mm
Changed lines of the file:
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@@
       (effects (font (size 1 1) (thickness 0.15)))
     )
-    (fp_text value "GLV_FUSE" (at 11.25 6) (layer "F.Fab")
+    (fp_text value "GLV_FUSE" (at 16.75 -2.5) (layer "F.Fab")
       (effects (font (size 1 1) (thickness 0.15)))
     )
@@
       (effects (font (size 1 1) (thickness 0.15)))
     )
-    (fp_text value "BUCK_SHUT" (at 5.08 5 90) (layer "F.Fab")
+    (fp_text value "BUCK_SHUT" (at 15.08 -2.5 180) (layer "F.Fab")
       (effects (font (size 1 1) (thickness 0.15)))
     )
@@
       (effects (font (size 1 1) (thickness 0.15)))
     )
-    (fp_text value "SPLIT_POWER" (at 2.54 5.08 90) (layer "F.Fab")
+    (fp_text value "SPLIT_POWER" (at 2.54 -7 90) (layer "F.Fab")
       (effects (font (size 1 1) (thickness 0.15)))
     )
@@
       (effects (font (size 1 1) (thickness 0.15)))
     )
-    (fp_text value "Fuse" (at 11.25 6) (layer "F.Fab")
+    (fp_text value "Fuse" (at 7.25 -0.5) (layer "F.Fab")
       (effects (font (size 1 1) (thickness 0.15)))
     )
@@
       (effects (font (size 1 1) (thickness 0.15)))
     )
-    (fp_text value "DC_CONVERTER" (at 5.08 5.08 90) (layer "F.Fab")
+    (fp_text value "DC_CONVERTER" (at 3.66 -9.5 90) (layer "F.Fab")
       (effects (font (size 1 1) (thickness 0.15)))
     )
@@
       (effects (font (size 1 1) (thickness 0.15)))
     )
-    (fp_text value "Fuse" (at 11.25 6) (layer "F.Fab")
-      (effects (font (size 1 1) (thickness 0.15)))
-    )
-    (fp_text user "${REFERENCE}" (at 11.25 4) (layer "F.Fab")
+    (fp_text value "Fuse" (at 11.25 4) (layer "F.Fab")
+      (effects (font (size 1 1) (thickness 0.15)))
+    )
+    (fp_text user "${REFERENCE}" (at 11.25 2.5) (layer "F.Fab")
       (effects (font (size 1 1) (thickness 0.15)))
     )
@@
     (property "Sheetname" "")
     (attr through_hole)
-    (fp_text reference "F13" (at 11.25 -6) (layer "F.SilkS")
+    (fp_text reference "F13" (at 17.75 0) (layer "F.SilkS")
       (effects (font (size 1 1) (thickness 0.15)))
     )
@@
       (effects (font (size 1 1) (thickness 0.15)))
     )
-    (fp_text value "VBAT" (at 2.54 5.08 90) (layer "F.Fab")
+    (fp_text value "VBAT" (at -2.46 -6 90) (layer "F.Fab")
       (effects (font (size 1 1) (thickness 0.15)))
     )
@@
     )
   )
+  (gr_rect (start 49.5 57) (end 144 152.5) (layer "Edge.Cuts") (width 0.1) (fill none))
   (segment (start 52.775489 121.970334) (end 59.805155 129) (width 2) (layer "B.Cu") (net 1))
   (segment (start 124.25 129) (end 128.25 133) (width 2) (layer "B.Cu") (net 1))
@@
   (segment (start 138 101.75) (end 138 90.95868) (width 2) (layer "B.Cu") (net 2))
   (segment (start 138 90.95868) (end 138.87868 90.08) (width 2) (layer "B.Cu") (net 2))
-  (segment (start 50.275969 123.00567) (end 50.275969 111.311531) (width 2) (layer "B.Cu") (net 3))
-  (segment (start 63.26981 135.999511) (end 50.275969 123.00567) (width 2) (layer "B.Cu") (net 3))
-  (segment (start 50.275969 111.311531) (end 55.5875 106) (width 2) (layer "B.Cu") (net 3))
   (segment (start 131.249511 134.750489) (end 130.000489 135.999511) (width 2) (layer "B.Cu") (net 3))
+  (segment (start 55.5875 106) (end 50.775969 110.811531) (width 1) (layer "B.Cu") (net 3))
+  (segment (start 50.775969 123.275969) (end 63.499511 135.999511) (width 1) (layer "B.Cu") (net 3))
   (segment (start 128.25 119) (end 131.249511 121.999511) (width 2) (layer "B.Cu") (net 3))
   (segment (start 131.249511 121.999511) (end 131.249511 134.750489) (width 2) (layer "B.Cu") (net 3))
-  (segment (start 130.000489 135.999511) (end 63.26981 135.999511) (width 2) (layer "B.Cu") (net 3))
+  (segment (start 64.000489 135.999511) (end 63.26981 135.999511) (width 2) (layer "B.Cu") (net 3))
+  (segment (start 130.000489 135.999511) (end 64.000489 135.999511) (width 2) (layer "B.Cu") (net 3))
+  (segment (start 63.499511 135.999511) (end 64.000489 135.999511) (width 1) (layer "B.Cu") (net 3))
+  (segment (start 50.775969 110.811531) (end 50.775969 123.275969) (width 1) (layer "B.Cu") (net 3))
   (segment (start 73.50805 60) (end 79.323721 60) (width 2) (layer "F.Cu") (net 4))
   (segment (start 55.5875 102) (end 52.775489 99.187989) (width 2) (layer "F.Cu") (net 4))
@@
   (via (at 91 68) (size 2) (drill 1) (layers "F.Cu" "B.Cu") (net 4))
   (segment (start 91 68) (end 110 68) (width 2) (layer "B.Cu") (net 4))
-  (segment (start 55.5875 98) (end 50.275969 92.688469) (width 2) (layer "B.Cu") (net 5))
-  (segment (start 50.275969 79.189175) (end 57.964176 71.500969) (width 2) (layer "B.Cu") (net 5))
+  (segment (start 50.775969 93.188469) (end 50.775969 78.689175) (width 1) (layer "B.Cu") (net 5))
+  (segment (start 50.775969 78.689175) (end 51.232572 78.232572) (width 1) (layer "B.Cu") (net 5))
   (segment (start 57.964176 71.500969) (end 122.750969 71.500969) (width 2) (layer "B.Cu") (net 5))
-  (segment (start 50.275969 92.688469) (end 50.275969 79.189175) (width 2) (layer "B.Cu") (net 5))
+  (segment (start 55.5875 98) (end 50.775969 93.188469) (width 1) (layer "B.Cu") (net 5))
+  (segment (start 51.232572 78.232572) (end 57.964176 71.500969) (width 2) (layer "B.Cu") (net 5))
   (segment (start 122.750969 71.500969) (end 128.25 77) (width 2) (layer "B.Cu") (net 5))
   (segment (start 80.49952 83.964665) (end 77.360334 80.825479) (width 2) (layer "B.Cu") (net 6))
@@
   (segment (start 101.25 59) (end 131 59) (width 2) (layer "F.Cu") (net 26))
   (segment (start 134 62) (end 134 66) (width 2) (layer "F.Cu") (net 26))
+  (zone (net 18) (net_name "GND") (layers F&B.Cu) (hatch edge 0.508)
+    (connect_pads (clearance 0.508))
+    (min_thickness 0.254) (filled_areas_thickness no)
+    (fill yes (thermal_gap 0.508) (thermal_bridge_width 0.508))
+    (polygon
+      (pts
+        (xy 143.5 151.5)
+        (xy 50 151.5)
+        (xy 50 57.5)
+        (xy 143.5 57.5)
+      )
+    )
+  )
 )
