File: EN-A0001-01001-AA - Placa de Fusíveis (BMS)/EN-A0001-01001-AA - Placa de Fusíveis (BMS).kicad_pcb (KiCad board)
At the start: 2 copper layers, 41 x 97 mm, 11 parts, among them J1 Conn_01x09_Male, J2 Conn_01x09_Male

Commit message: AA
Changed lines of the file:
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@@
     (property "Sheetname" "")
     (attr through_hole)
-    (fp_text reference "F1" (at 11.25 -6) (layer "F.SilkS")
+    (fp_text reference "F1" (at 16 -1) (layer "F.SilkS")
       (effects (font (size 1 1) (thickness 0.15)))
     )
@@
       (effects (font (size 1 1) (thickness 0.15)))
     )
-    (fp_text value "Fuse" (at 11.25 6) (layer "F.Fab")
+    (fp_text value "Fuse" (at 7 1) (layer "F.Fab")
       (effects (font (size 1 1) (thickness 0.15)))
     )
-    (fp_text user "${REFERENCE}" (at 11.25 4) (layer "F.Fab")
+    (fp_text user "${REFERENCE}" (at 15 0) (layer "F.Fab")
       (effects (font (size 1 1) (thickness 0.15)))
     )
